File: projects/secondlife-ups/hw/hw.kicad_sch (KiCad schematic)
At the start: 45 parts, among them J1 Screw_Terminal_01x03, J2 Screw_Terminal_01x02, J3 Screw_Terminal_01x02, J4 Screw_Terminal_01x02, J5 Screw_Terminal_01x02, J6 Tamiya, J7 Tamiya, J8 Tamiya, J9 Tamiya, K1 RM96Z-12-W, K2 SCB-1-M-1240, M1 AC PSU Fan, Q1 BC547, Q2 2N7000, SW1 SW_DIP_x01, SW2 SW_SPST_Temperature, SW3 SW_SPST_Temperature, U1 L7812, U2 LM339, U3 CC/CV Li-Ion charger, U4 XL4015 Module 12V/5A, U5 LM2596 Module 5V/3A

Commit message: rebuild
Parts:
- added U6: L7812, symbol Regulator_Linear:L7812
Connections:
- net +12V: now also J4.1 (Pin_1), J8.1 (Pin_1)
- net +24V: now also U6.1 (IN); no longer M1.1 (+)
- net +5V: no longer J4.1 (Pin_1), J8.1 (Pin_1)
- net GND: now also U6.2 (GND)
- new net: M1.1 (+), U6.3 (OUT)
Other:
- moved on the sheet: M1
Changed lines of the file:
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@@
-(kicad_sch (version 20210126) (generator eeschema)
+(kicad_sch (version 20210406) (generator eeschema)
   (paper "A4")
   (title_block
@@
   (symbol (lib_id "power:+24V") (at 31.75 129.54 90) (unit 1)
     (in_bom yes) (on_board yes) (fields_autoplaced)
-    (property "Reference" "#PWR?" (id 0) (at 35.56 129.54 0)
+    (property "Reference" "#PWR01" (id 0) (at 35.56 129.54 0)
       (effects (font (size 1.27 1.27)) hide)
     )
@@
     (pin "1")
   )
-  (symbol (lib_id "power:+24V") (at 57.15 106.68 0) (unit 1)
-    (in_bom yes) (on_board yes) (fields_autoplaced)
-    (property "Reference" "#PWR05" (id 0) (at 57.15 110.49 0)
-      (effects (font (size 1.27 1.27)) hide)
-    )
-    (property "Value" "+24V" (id 1) (at 57.15 102.87 0))
-    (property "Footprint" "" (id 2) (at 57.15 106.68 0)
-      (effects (font (size 1.27 1.27)) hide)
-    )
-    (property "Datasheet" "" (id 3) (at 57.15 106.68 0)
+  (symbol (lib_id "power:+24V") (at 49.53 107.95 90) (unit 1)
+    (in_bom yes) (on_board yes) (fields_autoplaced)
+    (property "Reference" "#PWR05" (id 0) (at 53.34 107.95 0)
+      (effects (font (size 1.27 1.27)) hide)
+    )
+    (property "Value" "+24V" (id 1) (at 45.72 108.5849 90)
+      (effects (font (size 1.27 1.27)) (justify left))
+    )
+    (property "Footprint" "" (id 2) (at 49.53 107.95 0)
+      (effects (font (size 1.27 1.27)) hide)
+    )
+    (property "Datasheet" "" (id 3) (at 49.53 107.95 0)
       (effects (font (size 1.27 1.27)) hide)
     )
@@
     (pin "1")
   )
-  (symbol (lib_id "power:+5V") (at 200.66 134.62 90) (unit 1)
-    (in_bom yes) (on_board yes) (fields_autoplaced)
-    (property "Reference" "#PWR031" (id 0) (at 204.47 134.62 0)
-      (effects (font (size 1.27 1.27)) hide)
-    )
-    (property "Value" "+5V" (id 1) (at 196.85 135.2549 90)
+  (symbol (lib_id "power:+12V") (at 200.66 134.62 90) (unit 1)
+    (in_bom yes) (on_board yes) (fields_autoplaced)
+    (property "Reference" "#PWR?" (id 0) (at 204.47 134.62 0)
+      (effects (font (size 1.27 1.27)) hide)
+    )
+    (property "Value" "+12V" (id 1) (at 196.85 135.2549 90)
       (effects (font (size 1.27 1.27)) (justify left))
     )
@@
     (pin "1")
   )
-  (symbol (lib_id "power:+5V") (at 243.84 133.35 90) (unit 1)
+  (symbol (lib_id "power:+12V") (at 243.84 133.35 90) (unit 1)
     (in_bom yes) (on_board yes) (fields_autoplaced)
     (property "Reference" "#PWR?" (id 0) (at 247.65 133.35 0)
       (effects (font (size 1.27 1.27)) hide)
     )
-    (property "Value" "+5V" (id 1) (at 240.03 133.9849 90)
+    (property "Value" "+12V" (id 1) (at 240.03 133.9849 90)
       (effects (font (size 1.27 1.27)) (justify left))
     )
@@
   (symbol (lib_id "power:+5V") (at 243.84 139.7 90) (unit 1)
     (in_bom yes) (on_board yes) (fields_autoplaced)
-    (property "Reference" "#PWR?" (id 0) (at 247.65 139.7 0)
+    (property "Reference" "#PWR047" (id 0) (at 247.65 139.7 0)
       (effects (font (size 1.27 1.27)) hide)
     )
@@
     (pin "1")
   )
-  (symbol (lib_id "power:GND") (at 57.15 119.38 0) (unit 1)
-    (in_bom yes) (on_board yes) (fields_autoplaced)
-    (property "Reference" "#PWR06" (id 0) (at 57.15 125.73 0)
-      (effects (font (size 1.27 1.27)) hide)
-    )
-    (property "Value" "GND" (id 1) (at 57.15 124.46 0))
-    (property "Footprint" "" (id 2) (at 57.15 119.38 0)
-      (effects (font (size 1.27 1.27)) hide)
-    )
-    (property "Datasheet" "" (id 3) (at 57.15 119.38 0)
+  (symbol (lib_id "power:GND") (at 57.15 115.57 0) (unit 1)
+    (in_bom yes) (on_board yes) (fields_autoplaced)
+    (property "Reference" "#PWR06" (id 0) (at 57.15 121.92 0)
+      (effects (font (size 1.27 1.27)) hide)
+    )
+    (property "Value" "GND" (id 1) (at 57.15 120.65 0))
+    (property "Footprint" "" (id 2) (at 57.15 115.57 0)
+      (effects (font (size 1.27 1.27)) hide)
+    )
+    (property "Datasheet" "" (id 3) (at 57.15 115.57 0)
       (effects (font (size 1.27 1.27)) hide)
     )
@@
     )
     (property "Datasheet" "" (id 3) (at 67.31 149.86 0)
+      (effects (font (size 1.27 1.27)) hide)
+    )
+    (pin "1")
+  )
+  (symbol (lib_id "power:GND") (at 77.47 107.95 90) (unit 1)
+    (in_bom yes) (on_board yes) (fields_autoplaced)
+    (property "Reference" "#PWR043" (id 0) (at 83.82 107.95 0)
+      (effects (font (size 1.27 1.27)) hide)
+    )
+    (property "Value" "GND" (id 1) (at 81.28 108.5849 90)
+      (effects (font (size 1.27 1.27)) (justify right))
+    )
+    (property "Footprint" "" (id 2) (at 77.47 107.95 0)
+      (effects (font (size 1.27 1.27)) hide)
+    )
+    (property "Datasheet" "" (id 3) (at 77.47 107.95 0)
       (effects (font (size 1.27 1.27)) hide)
     )
@@
     (pin "2")
   )
-  (symbol (lib_id "Motor:Fan") (at 57.15 114.3 0) (unit 1)
-    (in_bom yes) (on_board yes) (fields_autoplaced)
-    (property "Reference" "M1" (id 0) (at 62.23 112.3949 0)
-      (effects (font (size 1.27 1.27)) (justify left))
-    )
-    (property "Value" "AC PSU Fan" (id 1) (at 62.23 114.9349 0)
-      (effects (font (size 1.27 1.27)) (justify left))
-    )
-    (property "Footprint" "" (id 2) (at 57.15 114.046 0)
-      (effects (font (size 1.27 1.27)) hide)
-    )
-    (property "Datasheet" "~" (id 3) (at 57.15 114.046 0)
+  (symbol (lib_id "Motor:Fan") (at 72.39 107.95 90) (unit 1)
+    (in_bom yes) (on_board yes) (fields_autoplaced)
+    (property "Reference" "M1" (id 0) (at 71.12 100.33 90))
+    (property "Value" "AC PSU Fan" (id 1) (at 71.12 102.87 90))
+    (property "Footprint" "" (id 2) (at 72.136 107.95 0)
+      (effects (font (size 1.27 1.27)) hide)
+    )
+    (property "Datasheet" "~" (id 3) (at 72.136 107.95 0)
       (effects (font (size 1.27 1.27)) hide)
     )
@@
     (property "Datasheet" "https://www.onsemi.com/pub/Collateral/NDS7002A-D.PDF" (id 3) (at 172.72 66.04 0)
       (effects (font (size 1.27 1.27)) (justify left) hide)
+    )
+    (pin "1")
+    (pin "2")
+    (pin "3")
+  )
+  (symbol (lib_id "Regulator_Linear:L7812") (at 57.15 107.95 0) (unit 1)
+    (in_bom yes) (on_board yes) (fields_autoplaced)
+    (property "Reference" "U6" (id 0) (at 57.15 101.6 0))
+    (property "Value" "L7812" (id 1) (at 57.15 104.14 0))
+    (property "Footprint" "" (id 2) (at 57.785 111.76 0)
+      (effects (font (size 1.27 1.27) italic) (justify left) hide)
+    )
+    (property "Datasheet" "http://www.st.com/content/ccc/resource/technical/document/datasheet/41/4f/b3/b0/12/d4/47/88/CD00000444.pdf/files/CD00000444.pdf/jcr:content/translations/en.CD00000444.pdf" (id 3) (at 57.15 109.22 0)
+      (effects (font (size 1.27 1.27)) hide)
     )
     (pin "1")
@@
   )
   (symbol_instances
+    (path "/ca5f032d-583a-40ad-9a23-aaff2b0fe1af"
+      (reference "#PWR01") (unit 1) (value "+24V") (footprint "")
+    )
     (path "/774f4bbc-ce3c-46ee-b795-87f0975b9db6"
       (reference "#PWR02") (unit 1) (value "+BATT") (footprint "")
@@
       (reference "#PWR030") (unit 1) (value "GND") (footprint "")
     )
-    (path "/06edff92-9a1f-47ab-823d-d291a1d423da"
-      (reference "#PWR031") (unit 1) (value "+5V") (footprint "")
-    )
     (path "/96ee2358-ed81-450b-a240-808e745fc62c"
       (reference "#PWR032") (unit 1) (value "GND") (footprint "")
@@
       (reference "#PWR042") (unit 1) (value "GND") (footprint "")
     )
+    (path "/ea3bd7e6-9ee5-40b7-90f3-49278d91111f"
+      (reference "#PWR043") (unit 1) (value "GND") (footprint "")
+    )
     (path "/912fe703-6d7f-40b5-badc-a44a523f72f2"
       (reference "#PWR044") (unit 1) (value "GND") (footprint "")
@@
       (reference "#PWR046") (unit 1) (value "GND") (footprint "")
     )
-    (path "/7764210d-fab5-407e-a37a-5f989cbc19bd"
-      (reference "#PWR?") (unit 1) (value "+5V") (footprint "")
-    )
     (path "/c77b33da-72ff-4fe0-8093-73cc5ec77445"
-      (reference "#PWR?") (unit 1) (value "+5V") (footprint "")
-    )
-    (path "/ca5f032d-583a-40ad-9a23-aaff2b0fe1af"
-      (reference "#PWR?") (unit 1) (value "+24V") (footprint "")
+      (reference "#PWR047") (unit 1) (value "+5V") (footprint "")
+    )
+    (path "/44580b9b-f55a-43ca-89eb-12f2b881c30d"
+      (reference "#PWR?") (unit 1) (value "+12V") (footprint "")
+    )
+    (path "/eda41e28-e73b-4d63-bae8-37fd6e3dca5c"
+      (reference "#PWR?") (unit 1) (value "+12V") (footprint "")
     )
     (path "/45385ffc-dc77-4cef-8ae6-a1cb72f14691"
@@
       (reference "U5") (unit 1) (value "LM2596 Module 5V/3A") (footprint "")
     )
-  )
+    (path "/b460e2c4-983b-4f9e-89fe-2eae9c920c53"
+      (reference "U6") (unit 1) (value "L7812") (footprint "")
+    )
+  )
