File: projects/cell-precharger/cell-precharger.kicad/cell-precharger.kicad_pcb (KiCad board)
At the start: 2 copper layers, 22 x 18 mm, 10 parts, among them J1 Vin, J2 Vbat, U1 CJ431

Commit message: rebuild
Parts:
- moved REF** 2.06 mm to (155.0, 105.0)
Other:
- board size 22 x 18 mm -> 22 x 20 mm
Changed lines of the file:
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@@
       (outputformat 1)
       (mirror false)
-      (drillshape 1)
+      (drillshape 0)
       (scaleselection 1)
-      (outputdirectory "")
+      (outputdirectory "manuf-rev1/")
     )
   )
@@
   (net 5 "Net-(J2-Pad1)")
   (footprint "MountingHole:MountingHole_2.2mm_M2_ISO7380_Pad_TopBottom" (layer "F.Cu")
-    (at 155.5 107)
+    (at 155 105)
     (descr "Mounting Hole 2.2mm, M2, ISO7380")
     (tags "mounting hole 2.2mm m2 iso7380")
@@
     (fp_line (start -1.6 0.8) (end -1.6 -0.8) (layer "F.Fab") (width 0.1))
     (fp_line (start 1.6 -0.8) (end 1.6 0.8) (layer "F.Fab") (width 0.1))
-    (pad "1" smd roundrect locked (at -1.4625 0 180) (size 1.125 1.75) (layers "F.Cu" "F.Paste" "F.Mask") (roundrect_rratio 0.222222)
+    (pad "1" smd roundrect locked (at -1.4625 0 180) (size 1.125 1.75) (layers "F.Cu" "F.Paste" "F.Mask") (roundrect_rratio 0.2222222222)
       (net 5 "Net-(J2-Pad1)") (pintype "passive"))
-    (pad "2" smd roundrect locked (at 1.4625 0 180) (size 1.125 1.75) (layers "F.Cu" "F.Paste" "F.Mask") (roundrect_rratio 0.222222)
+    (pad "2" smd roundrect locked (at 1.4625 0 180) (size 1.125 1.75) (layers "F.Cu" "F.Paste" "F.Mask") (roundrect_rratio 0.2222222222)
       (net 4 "GND") (pintype "passive"))
     (model "${KICAD6_3DMODEL_DIR}/Resistor_SMD.3dshapes/R_1206_3216Metric.wrl"
@@
     (fp_line (start 5 2.2) (end 5 -1.6) (layer "F.Fab") (width 0.1))
     (fp_line (start -2.91 2.61) (end -0.41 2.61) (layer "F.Fab") (width 0.1))
-    (pad "1" thru_hole roundrect locked (at 0 0 270) (size 1.7 2) (drill 1) (layers *.Cu *.Mask) (roundrect_rratio 0.147059)
+    (pad "1" thru_hole roundrect locked (at 0 0 270) (size 1.7 2) (drill 1) (layers *.Cu *.Mask) (roundrect_rratio 0.1470588235)
       (net 3 "+5V") (pinfunction "Pin_1") (pintype "passive"))
     (pad "2" thru_hole oval locked (at 2.5 0 270) (size 1.7 2) (drill 1) (layers *.Cu *.Mask)
@@
     (fp_line (start 1.6 0.8) (end -1.6 0.8) (layer "F.Fab") (width 0.1))
     (fp_line (start -1.6 0.8) (end -1.6 -0.8) (layer "F.Fab") (width 0.1))
-    (pad "1" smd roundrect locked (at -1.4625 0) (size 1.125 1.75) (layers "F.Cu" "F.Paste" "F.Mask") (roundrect_rratio 0.222222)
+    (pad "1" smd roundrect locked (at -1.4625 0) (size 1.125 1.75) (layers "F.Cu" "F.Paste" "F.Mask") (roundrect_rratio 0.2222222222)
       (net 3 "+5V") (pintype "passive"))
-    (pad "2" smd roundrect locked (at 1.4625 0) (size 1.125 1.75) (layers "F.Cu" "F.Paste" "F.Mask") (roundrect_rratio 0.222222)
+    (pad "2" smd roundrect locked (at 1.4625 0) (size 1.125 1.75) (layers "F.Cu" "F.Paste" "F.Mask") (roundrect_rratio 0.2222222222)
       (net 5 "Net-(J2-Pad1)") (pintype "passive"))
     (model "${KICAD6_3DMODEL_DIR}/Resistor_SMD.3dshapes/R_1206_3216Metric.wrl"
@@
     (fp_line (start -2.91 2.61) (end -0.41 2.61) (layer "F.Fab") (width 0.1))
     (fp_line (start -2.5 2.2) (end 5 2.2) (layer "F.Fab") (width 0.1))
-    (pad "1" thru_hole roundrect locked (at 0 0 270) (size 1.7 2) (drill 1) (layers *.Cu *.Mask) (roundrect_rratio 0.147059)
+    (pad "1" thru_hole roundrect locked (at 0 0 270) (size 1.7 2) (drill 1) (layers *.Cu *.Mask) (roundrect_rratio 0.1470588235)
       (net 5 "Net-(J2-Pad1)") (pinfunction "Pin_1"))
     (pad "2" thru_hole oval locked (at 2.5 0 270) (size 1.7 2) (drill 1) (layers *.Cu *.Mask)
@@
     (property "Sheetname" "")
     (attr through_hole)
-    (fp_text reference "D1" (at -2 3) (layer "F.SilkS")
+    (fp_text reference "D1" (at -1 4) (layer "F.SilkS")
       (effects (font (size 1 1) (thickness 0.15)))
     )
@@
     )
   )
-  (gr_rect (start 137 103) (end 159 121) (layer "Edge.Cuts") (width 0.1) (fill none))
+  (gr_rect (start 137 101) (end 159 121) (layer "Edge.Cuts") (width 0.1) (fill none))
   (dimension (type aligned) (layer "Cmts.User")
     (pts (xy 137 103) (xy 159 103))
@@
   )
   (dimension (type aligned) (layer "Cmts.User")
-    (pts (xy 137 103) (xy 137 121))
+    (pts (xy 137 101) (xy 137 121))
     (height 3)
-    (gr_text "18.0000 mm" (at 132.85 112 90) (layer "Cmts.User")
+    (gr_text "20.0000 mm" (at 132.85 111 90) (layer "Cmts.User")
       (effects (font (size 1 1) (thickness 0.15)))
     )
@@
         (xy 158 120)
         (xy 138 120)
-        (xy 138 104)
-        (xy 158 104)
+        (xy 138 102)
+        (xy 158 102)
       )
     )

Commit message: rebuild
Routing:
- net Net-(D1-Pad1): track 19.0 -> 33.7 mm, vias 1 -> 0
Changed lines of the file:
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@@
   )
   (segment (start 151 106.25) (end 151 108) (width 0.25) (layer "F.Cu") (net 1))
+  (segment (start 141.2375 111.75) (end 139.75 111.75) (width 0.25) (layer "F.Cu") (net 1))
+  (segment (start 139.75 111.75) (end 139 111) (width 0.25) (layer "F.Cu") (net 1))
   (segment (start 146.5625 105.5) (end 150.25 105.5) (width 0.25) (layer "F.Cu") (net 1))
+  (segment (start 139 104.75) (end 140.25 103.5) (width 0.25) (layer "F.Cu") (net 1))
+  (segment (start 140.25 103.5) (end 146 103.5) (width 0.25) (layer "F.Cu") (net 1))
   (segment (start 150.25 105.5) (end 151 106.25) (width 0.25) (layer "F.Cu") (net 1))
-  (segment (start 145.55 116.0625) (end 146.5 115.1125) (width 0.25) (layer "F.Cu") (net 1))
+  (segment (start 147 105.0625) (end 146.5625 105.5) (width 0.25) (layer "F.Cu") (net 1))
   (segment (start 145 107.0625) (end 146.5625 105.5) (width 0.25) (layer "F.Cu") (net 1))
-  (segment (start 146.5 115.1125) (end 146.5 114.5) (width 0.25) (layer "F.Cu") (net 1))
-  (segment (start 146.5 114.5) (end 146.5 114.25) (width 0.25) (layer "F.Cu") (net 1))
-  (via (at 146.5 114.25) (size 0.8) (drill 0.4) (layers "F.Cu" "B.Cu") (net 1))
-  (segment (start 146.5 114.25) (end 151 109.75) (width 0.25) (layer "B.Cu") (net 1))
-  (segment (start 151 109.75) (end 151 108) (width 0.25) (layer "B.Cu") (net 1))
+  (segment (start 147 104.5) (end 147 105.0625) (width 0.25) (layer "F.Cu") (net 1))
+  (segment (start 146 103.5) (end 147 104.5) (width 0.25) (layer "F.Cu") (net 1))
+  (segment (start 139 111) (end 139 104.75) (width 0.25) (layer "F.Cu") (net 1))
+  (segment (start 145.55 116.0625) (end 141.2375 111.75) (width 0.25) (layer "F.Cu") (net 1))
   (segment (start 144 106) (end 143.5 106.5) (width 0.25) (layer "F.Cu") (net 2))
   (segment (start 145 108.9375) (end 147.5225 108.9375) (width 0.25) (layer "F.Cu") (net 2))
