File: hardware/toyota-corolla/avclan-interface/avclan-interface.kicad_sch (KiCad schematic)
At the start: 7 parts, among them J1 IEBus / AVC-LAN, J2 Conn_01x02_Pin, U1 LM339

Commit message: rebuild
Parts:
- removed J2: Conn_01x02_Pin, symbol Connector:Conn_01x02_Pin
- added J2 (x2): Conn_01x02_Pin, symbol Connector:Conn_01x02_Pin
- added U2: SN65176AP, Package_DIP:DIP-8_W7.62mm, symbol Interface_UART:SN75176AP
Connections:
- net +5V: now also U2.8 (VCC)
- net BUS_{n}: now also U2.7 (B)
- net GND: now also J2.1 (Pin_1), J2.1 (Pin_1), U2.5 (GND)
- net at R4.2, U1.2: now also J2.2 (Pin_2)
- new net: U2.2 (~{RE}), U2.3 (DE)
- new net: J2.2 (Pin_2), U2.4 (D)
- new net BUS_{p}: U2.6 (A)
